Commit message: throroughly broken - can't launch view_craft

File: craft_description/urdf/craft/craft_macro.ros2_control.xacro (robot description, xacro)
@@ -27,13 +27,13 @@
       </hardware>
       <joint name="${prefix}servo_joint">
-        <command_interface name="position">     <!-- Add/Remove interfaces as needed -->
+        <command_interface name="position"/>     <!-- Add/Remove interfaces as needed -->
           <!-- TODO try re-enabling -->
           <!-- <param name="min">-1</param>
           <param name="max">1</param> -->
-        </command_interface>
-        <state_interface name="position">
+        <!-- </command_interface> -->
+        <state_interface name="position"/>
           <!-- TODO try re-enabling -->
           <!-- <param name="initial_value">0.0</param> -->
-        </state_interface>
+        <!-- </state_interface> -->
       </joint>
       <!-- TODO implement, replace unrealistic position -->

File: craft_description/urdf/craft/craft_macro.xacro (robot description, xacro)
@@ -2,5 +2,5 @@
 <robot xmlns:xacro="http://wiki.ros.org/xacro">
   <xacro:include filename="$(find craft_description)/urdf/common.xacro" />
-  <xacro:arg name="square_hull" default="true"/>
+  <xacro:arg name="square_hull" default="false"/>
 	<xacro:if value="$(arg square_hull)">
 		<xacro:property name="chassis_length" value="0.5"/>
@@ -12,34 +12,16 @@
     <!-- base link -->
     <link name="${prefix}base_link">
-      <!-- Default inertial for Gazebo/Ingnition - copy and edit block from 'common.xacro'
-           to get more realistic behaviour-->
-      <!-- <xacro:default_inertial/>
-      <visual>
-        <origin xyz="0 0 0" rpy="0 0 0" />
-        <geometry>
-          <cylinder length="0.3" radius="0.3" /> -->
-<!--           <mesh filename="package://craft_description/meshes/craft/visual/base_link.stl" /> -->
-        <!-- </geometry>
-      </visual>
-      <collision>
-        <origin xyz="0 0 0" rpy="0 0 0" />
-        <geometry>
-          <cylinder length="0.3" radius="0.3" /> -->
-<!--           <mesh filename="package://craft_description/meshes/craft/collision/base_link.stl" /> -->
-        <!-- </geometry>
-      </collision> -->
     </link>
     <!-- link 1 -->
     <link name="${prefix}hullassm">
-      </xacro:unless>
       <visual>
         <origin xyz="0 0 0" rpy="0 0 0" />
         <geometry>
           <xacro:if value="$(arg square_hull)">
-					<box size="${chassis_length} ${chassis_width} ${chassis_height}" />
-				</xacro:if>
-				<xacro:unless value="$(arg square_hull)">
-          <mesh filename="package://craft_description/meshes/craft/visual/hullassm.stl" />
-        </xacro:unless>
+					  <box size="${chassis_length} ${chassis_width} ${chassis_height}" />
+				  </xacro:if>
+          <xacro:unless value="$(arg square_hull)">
+            <mesh filename="package://craft_description/meshes/craft/visual/hullassm.stl" />
+          </xacro:unless>
         </geometry>
         <material name="hullassm_material">
@@ -73,5 +55,5 @@
     </link>
     <gazebo reference="hullassm">
-        <material>Gazebo/DarkGrey  </material>
+      <material>Gazebo/DarkGrey</material>
     </gazebo>
     <!-- link 2 -->
@@ -100,5 +82,5 @@
     </link>
     <gazebo reference="propeller">
-        <material>Gazebo/Purple  </material>
+      <material>Gazebo/Purple</material>
     </gazebo>
     <!-- link 3 -->
@@ -127,5 +109,5 @@
     </link>
     <gazebo reference="topassm">
-        <material>Gazebo/White </material>
+      <material>Gazebo/White</material>
     </gazebo>
     <!-- link 4 -->
@@ -153,4 +135,7 @@
 		  </inertial>
     </link>
+    <gazebo reference="servocargoassm">
+      <material>Gazebo/Blue </material>
+    </gazebo>
     <!-- link 5 -->
     <link name="${prefix}rudder">
@@ -175,9 +160,6 @@
     </link>
     <gazebo reference="rudder">
-        <material>Gazebo/Yellow  </material>
-    </gazebo>
-    <!-- All-zero tool frame. This frame should correspond to the TOOL frame of the robot's controller.) -->
-    <link name="${prefix}tool0" />
-    <!-- tool link -->
+      <material>Gazebo/Yellow</material>
+    </gazebo>
     <!-- END LINKS -->
     <!-- JOINTS -->
@@ -200,5 +182,4 @@
       <child link="${prefix}propeller" />
       <axis xyz="0 0 1" />
-      <!-- <limit effort="0" lower="${radians(-180)}" upper="${radians(180)}" velocity="${radians(180)}" /> -->
     </joint>
     <!-- joint 3 -->
@@ -208,5 +189,4 @@
       <child link="${prefix}topassm" />
       <axis xyz="0 0 1" />
-      <!-- <limit effort="0" lower="${radians(-90)}" upper="${radians(180)}" velocity="${radians(270)}" /> -->
     </joint>
     <!-- joint 4 -->
@@ -216,29 +196,13 @@
       <child link="${prefix}servocargoassm" />
       <axis xyz="0 0 1" />
-      <!-- <limit effort="0" lower="${radians(-360)}" upper="${radians(360)}" velocity="${radians(360)}" /> -->
     </joint>
     <!-- joint 5 -->
     <joint name="${prefix}servo_joint" type="revolute">
-      <!-- NOTE - change r to -1.5708 if breaks -->
-      <origin xyz="3.43338e-16 -0.005715 0.074295" rpy="0 0 -1.03735e-13" />
+      <origin xyz="3.43338e-16 -0.005715 0.074295" rpy="-1.5708 0 -1.03735e-13" />
       <parent link="${prefix}servocargoassm" />
       <child link="${prefix}rudder" />
       <axis xyz="0 0 1" />
-      <!-- NOTE: change  lower="-1.5708" upper="1.5708" if breaks -->
-      <limit effort="0" lower="${radians(-90)}" upper="${radians(90)}" velocity="4.36" />
-    </joint>
-    <!-- joint 6 -->
-    <!-- <joint name="${prefix}joint6" type="revolute">
-      <origin xyz="0 0 0.1" rpy="0 ${-pi/2} 0" />
-      <parent link="${prefix}rudder" />
-      <child link="${prefix}link6" />
-      <axis xyz="0 0 1" />
-      <limit effort="0" lower="${radians(-360)}" upper="${radians(360)}" velocity="${radians(720)}" />
-    </joint> -->
-    <!-- tool frame - fixed frame -->
-    <joint name="${prefix}joint6-tool0" type="fixed">
-      <parent link="${prefix}link6" />
-      <child link="${prefix}tool0" />
-      <origin xyz="0 0 -0.115" rpy="0 ${-pi} ${-pi/2}" />
+      <!-- NOTE: future try lower="${radians(-90)}" upper="${radians(90)}" -->
+      <limit effort="0" lower="-1.5708" upper="1.5708" velocity="4.36" />
     </joint>
     <!-- END JOINTS -->

Commit message: split up to deal with gazebo_ros2_control ideosyncracies

File: craft_description/urdf/craft/craft_macro.ros2_control.xacro (robot description, xacro)
@@ -10,66 +10,46 @@
                simulation_controllers"
                >
-    <ros2_control name="${name}" type="system">
-      <hardware>
-        <xacro:if value="${use_mock_hardware}">
-          <plugin>mock_components/GenericSystem</plugin>
-          <param name="mock_sensor_commands">${mock_sensor_commands}</param>
-        </xacro:if>
-        <xacro:if value="${sim_gazebo_classic}">
+  <!-- real hardware plugin -->
+    <xacro:unless value="$(arg sim_gazebo_classic)">
+      <ros2_control name="${name}" type="system">
+        <hardware>
+          <!-- TODO implement real hardware interface here -->
           <plugin>gazebo_ros2_control/GazeboSystem</plugin>
-        </xacro:if>
-        <xacro:if value="${sim_gazebo}">
-          <plugin>ign_ros2_control/IgnitionSystem</plugin>
-        </xacro:if>
-        <xacro:unless value="${use_mock_hardware or sim_gazebo_classic or sim_gazebo}">
-          <plugin>robot_hardware_inteface/RobotHardwareInteface</plugin>
-        </xacro:unless>
-      </hardware>
-      <joint name="${prefix}servo_joint">
-        <command_interface name="position"/>     <!-- Add/Remove interfaces as needed -->
-          <!-- TODO try re-enabling -->
-          <!-- <param name="min">-1</param>
-          <param name="max">1</param> -->
-        <!-- </command_interface> -->
-        <state_interface name="position"/>
-          <!-- TODO try re-enabling -->
-          <!-- <param name="initial_value">0.0</param> -->
-        <!-- </state_interface> -->
-      </joint>
-      <!-- TODO implement, replace unrealistic position -->
-			<!-- TODO swap to actuator maybe?  -->
-      <joint name="${prefix}propeller_joint">
-        <command_interface name="velocity">     <!-- Add/Remove interfaces as needed -->
-          <param name="min">-10</param>
-          <param name="max">10</param>
-        </command_interface>
-        <state_interface name="position"/>
-        <state_interface name="velocity"/>
-      </joint>
-      <!-- Remove/change sensors as needed -->
-      <!-- <sensor name="tcp_fts_sensor">
-        <state_interface name="fx"/>
-        <state_interface name="fy"/>
-        <state_interface name="fz"/>
-        <state_interface name="tx"/>
-        <state_interface name="ty"/>
-        <state_interface name="tz"/> -->
-        <!-- Change sensors as needed -->
-        <!-- <param name="frame_id">tool0</param>
-        <param name="min_fx">-100</param>
-        <param name="max_fx">100</param>
-        <param name="min_fy">-100</param>
-        <param name="max_fy">100</param>
-        <param name="min_fz">-200</param>
-        <param name="max_fz">200</param>
-        <param name="min_tx">-10</param>
-        <param name="max_tx">10</param>
-        <param name="min_ty">-10</param>
-        <param name="max_ty">10</param>
-        <param name="min_tz">-15</param>
-        <param name="max_tz">15</param>
-      </sensor> -->
-    </ros2_control>
-    <xacro:if value="$(arg sim_gazebo_classic)">
+        </hardware>
+        <joint name="${prefix}servo_joint">
+          <command_interface name="position"/>     <!-- Add/Remove interfaces as needed -->
+          <state_interface name="position"/>
+        </joint>
+        <!-- TODO replace unrealistic position, swap to actuator maybe?  -->
+        <joint name="${prefix}propeller_joint">
+          <command_interface name="velocity">     <!-- Add/Remove interfaces as needed -->
+            <param name="min">-10</param>
+            <param name="max">10</param>
+          </command_interface>
+          <state_interface name="position"/>
+          <state_interface name="velocity"/>
+        </joint>
+      </ros2_control>
+    <xacro:unless>
+    <!-- gazebo hardware plugin -->
+    <xacro:if value="${sim_gazebo_classic}">
+      <ros2_control name="Gazebo${name}" type="system">
+        <hardware>
+          <plugin>gazebo_ros2_control/GazeboSystem</plugin>
+        </hardware>
+        <joint name="${prefix}servo_joint">
+          <command_interface name="position"/>     <!-- Add/Remove interfaces as needed -->
+          <state_interface name="position"/>
+        </joint>
+        <!-- TODO replace unrealistic position, swap to actuator maybe?  -->
+        <joint name="${prefix}propeller_joint">
+          <command_interface name="velocity">     <!-- Add/Remove interfaces as needed -->
+            <param name="min">-10</param>
+            <param name="max">10</param>
+          </command_interface>
+          <state_interface name="position"/>
+          <state_interface name="velocity"/>
+        </joint>
+      </ros2_control>
       <!-- Gazebo plugins -->
       <gazebo reference="world">
@@ -77,19 +57,10 @@
       <gazebo>
         <plugin filename="libgazebo_ros2_control.so" name="gazebo_ros2_control">
-          <parameters>${simulation_controllers}</parameters>
+          <!-- TODO chance back to passed in param to eliminate package name -->
+          <parameters>$(find craft_bringup)/config/craft_controllers.yaml</parameters>
+          <parameters>$(find craft_bringup)/config/gz_ros2_ctl_use_sim.yaml</parameters>
         </plugin>
       </gazebo>
-    </xacro:if>
-    <xacro:if value="$(arg sim_gazebo)">
-      <!-- Gazebo plugins -->
-      <gazebo reference="world">
-      </gazebo>
-      <gazebo>
-        <plugin filename="libign_ros2_control-system.so" name="ign_ros2_control::IgnitionROS2ControlPlugin">
-          <parameters>${simulation_controllers}</parameters>
-          <controller_manager_node_name>${prefix}controller_manager</controller_manager_node_name>
-        </plugin>
-      </gazebo>
-    </xacro:if>
+    <xacro:if>
   </xacro:macro>
 </robot>

Commit message: renamed files back to old way

File: craft_description/urdf/craft/craft_macro.ros2_control.xacro (robot description, xacro)
@@ -10,46 +10,66 @@
                simulation_controllers"
                >
-  <!-- real hardware plugin -->
-    <xacro:unless value="$(arg sim_gazebo_classic)">
-      <ros2_control name="${name}" type="system">
-        <hardware>
-          <!-- TODO implement real hardware interface here -->
+    <ros2_control name="${name}" type="system">
+      <hardware>
+        <xacro:if value="${use_mock_hardware}">
+          <plugin>mock_components/GenericSystem</plugin>
+          <param name="mock_sensor_commands">${mock_sensor_commands}</param>
+        </xacro:if>
+        <xacro:if value="${sim_gazebo_classic}">
           <plugin>gazebo_ros2_control/GazeboSystem</plugin>
-        </hardware>
-        <joint name="${prefix}servo_joint">
-          <command_interface name="position"/>     <!-- Add/Remove interfaces as needed -->
-          <state_interface name="position"/>
-        </joint>
-        <!-- TODO replace unrealistic position, swap to actuator maybe?  -->
-        <joint name="${prefix}propeller_joint">
-          <command_interface name="velocity">     <!-- Add/Remove interfaces as needed -->
-            <param name="min">-10</param>
-            <param name="max">10</param>
-          </command_interface>
-          <state_interface name="position"/>
-          <state_interface name="velocity"/>
-        </joint>
-      </ros2_control>
-    </xacro:unless>
-    <!-- gazebo hardware plugin -->
+        </xacro:if>
+        <xacro:if value="${sim_gazebo}">
+          <plugin>ign_ros2_control/IgnitionSystem</plugin>
+        </xacro:if>
+        <xacro:unless value="${use_mock_hardware or sim_gazebo_classic or sim_gazebo}">
+          <plugin>robot_hardware_inteface/RobotHardwareInteface</plugin>
+        </xacro:unless>
+      </hardware>
+      <joint name="${prefix}servo_joint">
+        <command_interface name="position"/>     <!-- Add/Remove interfaces as needed -->
+          <!-- TODO try re-enabling -->
+          <!-- <param name="min">-1</param>
+          <param name="max">1</param> -->
+        <!-- </command_interface> -->
+        <state_interface name="position"/>
+          <!-- TODO try re-enabling -->
+          <!-- <param name="initial_value">0.0</param> -->
+        <!-- </state_interface> -->
+      </joint>
+      <!-- TODO implement, replace unrealistic position -->
+			<!-- TODO swap to actuator maybe?  -->
+      <joint name="${prefix}propeller_joint">
+        <command_interface name="velocity">     <!-- Add/Remove interfaces as needed -->
+          <param name="min">-10</param>
+          <param name="max">10</param>
+        </command_interface>
+        <state_interface name="position"/>
+        <state_interface name="velocity"/>
+      </joint>
+      <!-- Remove/change sensors as needed -->
+      <!-- <sensor name="tcp_fts_sensor">
+        <state_interface name="fx"/>
+        <state_interface name="fy"/>
+        <state_interface name="fz"/>
+        <state_interface name="tx"/>
+        <state_interface name="ty"/>
+        <state_interface name="tz"/> -->
+        <!-- Change sensors as needed -->
+        <!-- <param name="frame_id">tool0</param>
+        <param name="min_fx">-100</param>
+        <param name="max_fx">100</param>
+        <param name="min_fy">-100</param>
+        <param name="max_fy">100</param>
+        <param name="min_fz">-200</param>
+        <param name="max_fz">200</param>
+        <param name="min_tx">-10</param>
+        <param name="max_tx">10</param>
+        <param name="min_ty">-10</param>
+        <param name="max_ty">10</param>
+        <param name="min_tz">-15</param>
+        <param name="max_tz">15</param>
+      </sensor> -->
+    </ros2_control>
     <xacro:if value="$(arg sim_gazebo_classic)">
-      <ros2_control name="Gazebo${name}" type="system">
-        <hardware>
-          <plugin>gazebo_ros2_control/GazeboSystem</plugin>
-        </hardware>
-        <joint name="${prefix}servo_joint">
-          <command_interface name="position"/>     <!-- Add/Remove interfaces as needed -->
-          <state_interface name="position"/>
-        </joint>
-        <!-- TODO replace unrealistic position, swap to actuator maybe?  -->
-        <joint name="${prefix}propeller_joint">
-          <command_interface name="velocity">     <!-- Add/Remove interfaces as needed -->
-            <param name="min">-10</param>
-            <param name="max">10</param>
-          </command_interface>
-          <state_interface name="position"/>
-          <state_interface name="velocity"/>
-        </joint>
-      </ros2_control>
       <!-- Gazebo plugins -->
       <gazebo reference="world">
@@ -57,7 +77,16 @@
       <gazebo>
         <plugin filename="libgazebo_ros2_control.so" name="gazebo_ros2_control">
-          <!-- TODO chance back to passed in param to eliminate package name -->
-          <parameters>$(find craft_bringup)/config/craft_controllers.yaml</parameters>
-          <parameters>$(find craft_bringup)/config/gz_ros2_ctl_use_sim.yaml</parameters>
+          <parameters>${simulation_controllers}</parameters>
+        </plugin>
+      </gazebo>
+    </xacro:if>
+    <xacro:if value="$(arg sim_gazebo)">
+      <!-- Gazebo plugins -->
+      <gazebo reference="world">
+      </gazebo>
+      <gazebo>
+        <plugin filename="libign_ros2_control-system.so" name="ign_ros2_control::IgnitionROS2ControlPlugin">
+          <parameters>${simulation_controllers}</parameters>
+          <controller_manager_node_name>${prefix}controller_manager</controller_manager_node_name>
         </plugin>
       </gazebo>
