Commit message: switched to using args because params were being annoying

File: craft_description/urdf/craft.urdf.xacro (robot description, xacro)
@@ -17,11 +17,3 @@
     <origin xyz="0 0 0" rpy="0 0 0" />          <!-- position robot in the world -->
   </xacro:craft>
-  <xacro:craft_ros2_control
-    name="craft"
-    prefix="$(arg prefix)"
-    use_mock_hardware="$(arg use_mock_hardware)"
-    mock_sensor_commands="$(arg mock_sensor_commands)"
-    sim_gazebo_classic="$(arg sim_gazebo_classic)"
-    sim_gazebo="$(arg sim_gazebo)"
-    simulation_controllers="$(arg simulation_controllers)" />
 </robot>

File: craft_description/urdf/craft/craft_macro.ros2_control.xacro (robot description, xacro)
@@ -1,26 +1,24 @@
 <?xml version="1.0" encoding="UTF-8"?>
 <robot xmlns:xacro="http://wiki.ros.org/xacro">
-  <xacro:macro name="craft_ros2_control" params="
-               name
-               prefix
-               use_mock_hardware:=^|false
-               mock_sensor_commands:=^|false
-               sim_gazebo_classic:=^|false
-               sim_gazebo:=^|false
-               simulation_controllers"
-               >
-    <ros2_control name="${name}" type="system">
+  <xacro:arg name="name" default="craft"/>
+  <xacro:arg name="prefix" default=""/>
+  <xacro:arg name="use_mock_hardware" default="false"/>
+  <xacro:arg name="mock_sensor_commands" default="false"/>
+  <xacro:arg name="sim_gazebo_classic" default="false"/>
+  <xacro:arg name="sim_gazebo" default="false"/>
+  <xacro:arg name="real_hardware" default="false"/>
+    <ros2_control name="$(arg name)" type="system">
       <hardware>
-        <xacro:if value="${use_mock_hardware}">
+        <xacro:if value="$(arg use_mock_hardware)">
           <plugin>mock_components/GenericSystem</plugin>
-          <param name="mock_sensor_commands">${mock_sensor_commands}</param>
+          <param name="mock_sensor_commands">$(arg mock_sensor_commands)</param>
         </xacro:if>
-        <xacro:if value="${sim_gazebo_classic}">
+        <xacro:if value="$(arg sim_gazebo_classic)">
           <plugin>gazebo_ros2_control/GazeboSystem</plugin>
         </xacro:if>
-        <xacro:if value="${sim_gazebo}">
+        <xacro:if value="$(arg sim_gazebo)">
           <plugin>ign_ros2_control/IgnitionSystem</plugin>
         </xacro:if>
-        <xacro:unless value="${use_mock_hardware or sim_gazebo_classic or sim_gazebo}">
+        <xacro:if value="$(arg real_hardware)">
           <plugin>craft_hardware/CraftHardware</plugin>
           <param name="srv_name">servo_joint</param>
@@ -30,7 +28,7 @@
           <param name="srv_min_pulse_width_us">650</param>
           <param name="srv_max_pulse_width_us">2500</param>
-        </xacro:unless>
+        </xacro:if>
       </hardware>
-      <joint name="${prefix}servo_joint">
+      <joint name="$(arg prefix)servo_joint">
         <command_interface name="position"/>     <!-- Add/Remove interfaces as needed -->
           <!-- TODO try re-enabling -->
@@ -38,18 +36,22 @@
           <param name="max">1</param> -->
         <!-- </command_interface> -->
-        <state_interface name="position"/>
+        <state_interface name="position">
           <!-- TODO try re-enabling -->
-          <!-- <param name="initial_value">0.0</param> -->
-        <!-- </state_interface> -->
+          <param name="initial_value">0.0</param>
+        </state_interface>
       </joint>
       <!-- TODO implement, replace unrealistic position -->
 			<!-- TODO swap to actuator maybe?  -->
-      <joint name="${prefix}propeller_joint">
+      <joint name="$(arg prefix)propeller_joint">
         <command_interface name="velocity">     <!-- Add/Remove interfaces as needed -->
           <param name="min">-10</param>
           <param name="max">10</param>
         </command_interface>
-        <state_interface name="position"/>
-        <state_interface name="velocity"/>
+        <state_interface name="position">
+          <param name="initial_value">0.0</param>
+        </state_interface>
+        <state_interface name="velocity">
+          <param name="initial_value">0.0</param>
+        </state_interface>
       </joint>
       <!-- Remove/change sensors as needed -->
@@ -83,5 +85,5 @@
       <gazebo>
         <plugin filename="libgazebo_ros2_control.so" name="gazebo_ros2_control">
-          <parameters>${simulation_controllers}</parameters>
+          <parameters>$(find craft_bringup)/config/craft_controllers.yaml</parameters>
         </plugin>
       </gazebo>
@@ -93,9 +95,8 @@
       <gazebo>
         <plugin filename="libign_ros2_control-system.so" name="ign_ros2_control::IgnitionROS2ControlPlugin">
-          <parameters>${simulation_controllers}</parameters>
-          <controller_manager_node_name>${prefix}controller_manager</controller_manager_node_name>
+          <parameters>$(find craft_bringup)/config/craft_controllers.yaml</parameters>
+          <controller_manager_node_name>$(arg prefix)controller_manager</controller_manager_node_name>
         </plugin>
       </gazebo>
     </xacro:if>
-  </xacro:macro>
 </robot>

Commit message: Revert "switched to using args because params were being annoying"
This reverts commit 4a4a4c484e58504f74fa4033bf2d5b28237a746d.

File: craft_description/urdf/craft.urdf.xacro (robot description, xacro)
@@ -17,3 +17,11 @@
     <origin xyz="0 0 0" rpy="0 0 0" />          <!-- position robot in the world -->
   </xacro:craft>
+  <xacro:craft_ros2_control
+    name="craft"
+    prefix="$(arg prefix)"
+    use_mock_hardware="$(arg use_mock_hardware)"
+    mock_sensor_commands="$(arg mock_sensor_commands)"
+    sim_gazebo_classic="$(arg sim_gazebo_classic)"
+    sim_gazebo="$(arg sim_gazebo)"
+    simulation_controllers="$(arg simulation_controllers)" />
 </robot>

File: craft_description/urdf/craft/craft_macro.ros2_control.xacro (robot description, xacro)
@@ -1,24 +1,26 @@
 <?xml version="1.0" encoding="UTF-8"?>
 <robot xmlns:xacro="http://wiki.ros.org/xacro">
-  <xacro:arg name="name" default="craft"/>
-  <xacro:arg name="prefix" default=""/>
-  <xacro:arg name="use_mock_hardware" default="false"/>
-  <xacro:arg name="mock_sensor_commands" default="false"/>
-  <xacro:arg name="sim_gazebo_classic" default="false"/>
-  <xacro:arg name="sim_gazebo" default="false"/>
-  <xacro:arg name="real_hardware" default="false"/>
-    <ros2_control name="$(arg name)" type="system">
+  <xacro:macro name="craft_ros2_control" params="
+               name
+               prefix
+               use_mock_hardware:=^|false
+               mock_sensor_commands:=^|false
+               sim_gazebo_classic:=^|false
+               sim_gazebo:=^|false
+               simulation_controllers"
+               >
+    <ros2_control name="${name}" type="system">
       <hardware>
-        <xacro:if value="$(arg use_mock_hardware)">
+        <xacro:if value="${use_mock_hardware}">
           <plugin>mock_components/GenericSystem</plugin>
-          <param name="mock_sensor_commands">$(arg mock_sensor_commands)</param>
+          <param name="mock_sensor_commands">${mock_sensor_commands}</param>
         </xacro:if>
-        <xacro:if value="$(arg sim_gazebo_classic)">
+        <xacro:if value="${sim_gazebo_classic}">
           <plugin>gazebo_ros2_control/GazeboSystem</plugin>
         </xacro:if>
-        <xacro:if value="$(arg sim_gazebo)">
+        <xacro:if value="${sim_gazebo}">
           <plugin>ign_ros2_control/IgnitionSystem</plugin>
         </xacro:if>
-        <xacro:if value="$(arg real_hardware)">
+        <xacro:unless value="${use_mock_hardware or sim_gazebo_classic or sim_gazebo}">
           <plugin>craft_hardware/CraftHardware</plugin>
           <param name="srv_name">servo_joint</param>
@@ -28,7 +30,7 @@
           <param name="srv_min_pulse_width_us">650</param>
           <param name="srv_max_pulse_width_us">2500</param>
-        </xacro:if>
+        </xacro:unless>
       </hardware>
-      <joint name="$(arg prefix)servo_joint">
+      <joint name="${prefix}servo_joint">
         <command_interface name="position"/>     <!-- Add/Remove interfaces as needed -->
           <!-- TODO try re-enabling -->
@@ -36,22 +38,18 @@
           <param name="max">1</param> -->
         <!-- </command_interface> -->
-        <state_interface name="position">
+        <state_interface name="position"/>
           <!-- TODO try re-enabling -->
-          <param name="initial_value">0.0</param>
-        </state_interface>
+          <!-- <param name="initial_value">0.0</param> -->
+        <!-- </state_interface> -->
       </joint>
       <!-- TODO implement, replace unrealistic position -->
 			<!-- TODO swap to actuator maybe?  -->
-      <joint name="$(arg prefix)propeller_joint">
+      <joint name="${prefix}propeller_joint">
         <command_interface name="velocity">     <!-- Add/Remove interfaces as needed -->
           <param name="min">-10</param>
           <param name="max">10</param>
         </command_interface>
-        <state_interface name="position">
-          <param name="initial_value">0.0</param>
-        </state_interface>
-        <state_interface name="velocity">
-          <param name="initial_value">0.0</param>
-        </state_interface>
+        <state_interface name="position"/>
+        <state_interface name="velocity"/>
       </joint>
       <!-- Remove/change sensors as needed -->
@@ -85,5 +83,5 @@
       <gazebo>
         <plugin filename="libgazebo_ros2_control.so" name="gazebo_ros2_control">
-          <parameters>$(find craft_bringup)/config/craft_controllers.yaml</parameters>
+          <parameters>${simulation_controllers}</parameters>
         </plugin>
       </gazebo>
@@ -95,8 +93,9 @@
       <gazebo>
         <plugin filename="libign_ros2_control-system.so" name="ign_ros2_control::IgnitionROS2ControlPlugin">
-          <parameters>$(find craft_bringup)/config/craft_controllers.yaml</parameters>
-          <controller_manager_node_name>$(arg prefix)controller_manager</controller_manager_node_name>
+          <parameters>${simulation_controllers}</parameters>
+          <controller_manager_node_name>${prefix}controller_manager</controller_manager_node_name>
         </plugin>
       </gazebo>
     </xacro:if>
+  </xacro:macro>
 </robot>
